Commit message: path planning

File: install/warehouse_robot/share/warehouse_robot/urdf/warehouse_amr.urdf (robot description, URDF)
Before this commit: robot warehouse_amr, 13 links, 12 joints
Joints:
- joint lidar_joint: origin xyz=-0.25 0 0.115 rpy=0 0 0 -> xyz=0.25 0 0.115 rpy=0 0 0

Commit message: rviz2 showing robot

File: install/warehouse_robot/share/warehouse_robot/urdf/warehouse_amr.urdf (robot description, URDF)
Before this commit: robot warehouse_amr, 13 links, 12 joints
Joints:
- joint caster_front_joint: origin xyz=0.28 0 -0.085 rpy=0 0 0 -> xyz=0 0 0.14 rpy=0 0 0
